Commit message: poignet axe 5 BLDC : driver Python, pont ros2_control, firmware SimpleFOC (US-027..030)
Travail developpe les 2026-09-12/13 SANS le materiel (poignet non monte). Rien ne
change tant que wrist:=servo (defaut) : l'URDF servo genere est identique octet pour
octet, une valeur de wrist invalide est une erreur.

- src/roby_wrist_bldc (nouveau) : protocole serie, generateur de consigne limite en
  vitesse/acceleration, detection du port, driver (thread lecteur, etat thread-safe,
  reconnexion, recalage au nid par Z, gestion des defauts), carte simulee, noeud ROS
  (/roby/wrist_bldc/{command,state,fault,status} + services), CLI, banc T1..T11,
  regle udev, config, launch.
- roby_hardware : JointType::BLDC, fil de publication de la consigne, retour d'etat
  du noeud BLDC, exclu du watchdog d'ecart ; xacro wrist:=servo|bldc ;
  robot_control.launch.py : argument wrist.
- pc_moveit.launch.py : argument wrist (joint_5 limite a 0,5 rad/s en bldc).
- firmware/wrist_bldc_simplefoc : firmware B-G431B-ESC1 (copie de
  ~/Documents/PlatformIO/Projects/test_bldc, md5 identique) + README (defauts F1-F7).
- tests : 67 tests roby_wrist_bldc (carte simulee), 3 tests du pont (roby_hardware).

Corrige pendant la revue du 2026-09-13 :
- DEFAUT DE SECURITE : apres reset_fault / enable / recalibrate_nest, le verrou qui
  ignore la vieille consigne de maintien n'etait pose qu'au tick de publication
  suivant (<= 20 ms, plus sous charge). Une consigne arrivee entre-temps etait suivie
  et l'axe repartait vers l'obstacle (jusqu'a 0,4 rad en test). Verrou pose AVANT de
  re-autoriser le mouvement + transition verifiee a chaque consigne. Test de
  regression deterministe (echoue 3/3 sans la correction).
- tests du noeud : attente de conditions en maintenant la consigne (attendre sans
  publier declenchait le timeout de commande) ; domaine DDS surchargeable
  (ROBY_TEST_DOMAIN_ID, 42/43 refuses). 12 series paralleles isolees : 67/67.
- limiter.py : le depassement ~v^2/2a a l'arret net d'une rampe est documente.

Verifie : pytest 67/67 (x12 en parallele), black, ruff, mypy propres.
LIMITE : jamais essaye sur la carte reelle ni le moteur (US-031).

Co-Authored-By: Claude Opus 5 (1M context) <noreply@anthropic.com>
Claude-Session: https://claude.ai/code/session_01DjFuuNz2SS97Ye1HUrD4PN

File: src/roby_hardware/config/roby_hardware_steppers_only.ros2_control.xacro (robot description, xacro)
@@ -5,7 +5,14 @@
   joints 4-5 = mock (servo/brushless not tested yet)
   coupling axes 2/3 ENABLED
+  wrist : actionneur de l'axe 5
+    servo (defaut) = servo provisoire PCA9685 CH1 (poignet actuel)
+    bldc           = LA8308 + cycloidal 20:1 via carte B-G431B-ESC1 et le noeud
+                     roby_wrist_bldc (spec-poignet-axe5-bldc, ADR-004)
 -->
 <robot xmlns:xacro="http://www.ros.org/wiki/xacro">
-    <xacro:macro name="roby_hardware_ros2_control" params="name initial_positions_file use_mock:=false">
+    <xacro:macro name="roby_hardware_ros2_control" params="name initial_positions_file use_mock:=false wrist:=servo">
+        <xacro:if value="${wrist not in ['servo', 'bldc']}">
+            <xacro:property name="_wrist_error" value="${xacro.fatal('wrist doit valoir servo ou bldc, recu : ' + wrist)}" lazy_eval="false"/>
+        </xacro:if>
         <xacro:property name="initial_positions" value="${xacro.load_yaml(initial_positions_file)['initial_positions']}"/>
         <ros2_control name="${name}" type="system">
@@ -48,4 +55,5 @@
                     <param name="joint_4_servo_offset_deg">135.0</param>
                     <param name="joint_4_inverted">false</param>
+                    <xacro:if value="${wrist == 'servo'}">
                     <!-- Axis 5: servo provisoire (brushless non monte), PCA9685 CH1 -->
                     <param name="joint_5_type">servo</param>
@@ -56,4 +64,15 @@
                     <param name="joint_5_servo_offset_deg">41.3</param>
                     <param name="joint_5_inverted">true</param>
+                    </xacro:if>
+                    <xacro:if value="${wrist == 'bldc'}">
+                    <!-- Axis 5: BLDC LA8308 + cycloidal 20:1, carte B-G431B-ESC1 (USB).
+                         Le plugin relaie consigne/mesure ; le noeud wrist_bldc parle a
+                         la carte (rampe, butees, securite). PCA9685 CH1 libre. -->
+                    <param name="joint_5_type">bldc</param>
+                    <param name="joint_5_bldc_command_topic">/roby/wrist_bldc/command</param>
+                    <param name="joint_5_bldc_state_topic">/roby/wrist_bldc/state</param>
+                    <param name="joint_5_bldc_state_timeout_s">0.2</param>
+                    <param name="joint_5_bldc_wait_on_activate_s">8.0</param>
+                    </xacro:if>
                     <!-- I2C config (unused but kept for init) -->
                     <param name="i2c_bus">/dev/i2c-1</param>

File: src/roby_hardware/config/roby_motor1_test.urdf.xacro (robot description, xacro)
@@ -6,8 +6,10 @@
 <robot xmlns:xacro="http://www.ros.org/wiki/xacro" name="neuroneimitationcarote">
     <xacro:arg name="initial_positions_file" default="$(find roby_hardware)/config/initial_positions.yaml" />
+    <!-- Axe 5 : servo (poignet actuel, defaut) ou bldc (nouveau poignet) -->
+    <xacro:arg name="wrist" default="servo" />
     <!-- Import robot URDF -->
     <xacro:include filename="$(find neuroneimitationcarote_description)/urdf/robot.urdf.xacro" />
     <!-- Import steppers ros2_control config (joints 1-3 real, 4-5 mock) -->
     <xacro:include filename="$(find roby_hardware)/config/roby_hardware_steppers_only.ros2_control.xacro" />
-    <xacro:roby_hardware_ros2_control name="RobySystem" initial_positions_file="$(arg initial_positions_file)" use_mock="false"/>
+    <xacro:roby_hardware_ros2_control name="RobySystem" initial_positions_file="$(arg initial_positions_file)" use_mock="false" wrist="$(arg wrist)"/>
 </robot>
