Commit message: Modèle: butée axe 2 élargie, collision link_2/link_4 désactivée, package roby_environments
- joint_2: limite -1.0/1.2 -> -1.6/2.1 (URDF robot.urdf.xacro)
- SRDF: disable_collisions link_2 <-> link_4 (reason User)
- Nouveau package roby_environments: environnements de collision chargeables
  dans la planning scene MoveIt (scene_loader: box/cylinder/sphere + couleurs ;
  environnement atelier_actuel.yaml mesuré).

Co-Authored-By: Claude Opus 4.8 (1M context) <noreply@anthropic.com>

File: src/neuroneimitationcarote_description/urdf/robot.urdf.xacro (robot description, xacro)
@@ -76,5 +76,5 @@
     <origin xyz="0.024031 0 0.202992" rpy="0 0 0"/>
     <axis xyz="0 1 0"/>
-    <limit lower="-1.0" upper="1.2" effort="20.0" velocity="1.0"/>
+    <limit lower="-1.6" upper="2.1" effort="20.0" velocity="1.0"/>
     <dynamics damping="0.5" friction="0.1" acceleration="1.0"/>
   </joint>

Commit message: Bras guide en joystick, cuisine 3D et zone de dataset
Bras guide (US-017/018/019) — ids attribues, calibration, mode joystick

Les 6 servos portent leurs identifiants et leurs bornes sont relevees. Le noeud
`leader_node` publie l'etat du bras et gere son couple ; il est seul proprietaire
du bus (verrou exclusif), demarre couple coupe et le coupe a l'arret.

Le leader ne commande plus une position mais une VITESSE : chaque axe est rappele
vers son zero avec un couple croissant, l'ecart devenant une consigne de vitesse.
Cela regle du meme coup l'affaissement du bras (le rappel le tient) et les 124 deg
de course inatteignables en correspondance 1:1.

Trois pieges ont ete corriges dans le driver, chacun verrouille par un test :
- le code retour de l'ecriture d'ID ment (le servo repond avec le NOUVEL id) ;
- activer le couple sans figer la cible fait sauter le servo vers une pose perimee ;
- un log a severite variable fait planter rclpy — au pire moment, la coupure du mode.

Les signes de correspondance avaient tous ete DEDUITS par calcul, et tous etaient
faux. Ce sont les essais qui les ont fixes ; les tests le documentent pour qu'on ne
les "recorrige" pas depuis un raisonnement geometrique.

Cuisine — import du plan 3D de l'equipe Le NIC

`roby_usd_to_environment.py` convertit la geometrie de collision USD en environnement
roby_environments : 35 obstacles colores (couleurs dominantes lues dans les materiaux
Sweet Home 3D), exprimes dans le repere de la base du robot.

Le support du robot demandait deux traitements : son sommet est rabote sous la base
(il PORTE le robot, leur contact n'est pas une collision et bloquait toute pose), et
une rotation de -90 deg aligne la scene sur le repere robot. Cette rotation est
confirmee par deux sources independantes qui coincident alors a 3 mm.

Nid recale et maillage recentre

Le nid passe a [1.5627, 0.9179, 0.4520, 0, 0.2009] pour que le changeur d'outil
tombe dans son logement, face basse horizontale. Les trajectoires sont decalees du
meme ecart : en boucle ouverte un angle est un compteur de pas, donc re-etiqueter le
nid sans les decaler inverserait le premier segment de sortie.

Le maillage de la section 4 etait stocke a 4 m de son origine, compense dans l'URDF.
RViz calculait donc son volume englobant a 4 m et l'eliminait du rendu selon l'angle
de vue. Il est recentre, l'URDF n'a plus besoin de compensation.

Zone de dataset dans la cuisine

Zone 45x46 cm bornee par la structure sous le robot, le refrigerateur et la plaque
de cuisson, avec 10 cm de marge. Hauteur de prise a +0,2551 m, soit la meme distance
a la surface que sur l'ancienne table. 90 % de la zone est atteignable en prise
verticale ; le script rejette deja les points qui ne le sont pas.

Restent a traiter avant toute collecte : le point de depose D est encore dans
l'ancienne zone (il deposerait au-dessus de la plaque), et la correction
d'inclinaison de table est desactivee car calibree sur l'atelier.

59 tests, sans ROS ni materiel.

Co-Authored-By: Claude Opus 5 (1M context) <noreply@anthropic.com>
Claude-Session: https://claude.ai/code/session_01FzZPeDj7ZhzKtGBWkvZXzU

File: src/neuroneimitationcarote_description/urdf/robot.urdf.xacro (robot description, xacro)
@@ -144,5 +144,5 @@
   <link name="link_4">
     <visual>
-      <origin xyz="-3.94046 0.0 0.0" rpy="0 0 0"/>
+      <origin xyz="0 0 0" rpy="0 0 0"/>
       <geometry>
         <mesh filename="package://neuroneimitationcarote_description/meshes/visual/section4_maillage.stl"

Commit message: URDF mesuree + cinematique a source unique (ADR-005)
La description du bras a ete re-mesuree et corrigee. A pose articulaire identique, la
pince se deplace de 125 mm au nid : l'epaule descend de 5,87 cm et l'origine de joint_5
quitte l'axe de roulis de joint_4 en prenant 9,9 cm en z.

Le probleme n'etait pas l'URDF mais sa duplication : la meme chaine cinematique etait
recopiee a la main dans trois fichiers Python sans aucun lien avec elle --
roby_tool_pickup (teleop, oracle, inference, prise d'outil), roby_oracle (que la GARDE
importe pour son plancher et son anti-collision) et visual_servo_node. Remplacer la seule
URDF aurait laisse la garde proteger le bras avec une geometrie fausse de plus de 10 cm,
sans que rien ne le signale.

- tools/pc/roby_cinematique.py : lit la chaine base_link -> link_gripper dans l'URDF du
  workspace en service et expose fkT / fk_pos / fk_poignet / jac / LIMITS. Il leve si
  l'URDF manque : une cinematique de repli silencieuse serait le defaut qu'on supprime.
- les trois copies l'importent et ne portent plus aucune constante geometrique.
- porte "geometrie" dans roby_gates : l'URDF publiee par la stack doit avoir la meme
  chaine que celle du depot. Une machine non redeployee devient visible avant tout
  mouvement, au lieu de rester silencieuse. Elle protege aussi tout programme qui passe
  par porte_stack (jog, sortie du nid, oracle, garde).
- tests : relecture independante de l'URDF, coherence FK/jacobienne, et refus qu'une
  origine mesuree ou une butee reapparaisse en dur dans l'un des trois fichiers.

Consequence mesuree sur la teleop : joint_4 deplace maintenant le centre du poignet
d'environ 10 cm/rad. Le bras guide partageant la description, le robot reproduit ce
deplacement a 1:1 -- ce n'est pas une derive, mais l'hypothese qui justifiait de piloter
ce point ne tient plus. Les deux tests qui affirmaient l'invariance sont reecrits pour
dire ce qui est vrai ; le choix du point commande est a reprendre (ADR-005).

⚠️ Toutes les constantes cartesiennes mesurees dans l'ancien repere sont fausses
(Z_SURFACE_CUISINE, Z_PICK_CUISINE, TABLE_PHYS, inclinaison, planchers garde et teleop) :
elles doivent etre re-mesurees sur le robot avant toute collecte.

Co-Authored-By: Claude Opus 5 (1M context) <noreply@anthropic.com>
Claude-Session: https://claude.ai/code/session_0187Ttw7QawW3jcZqaeAZY1B

File: src/neuroneimitationcarote_description/urdf/robot.urdf.xacro (robot description, xacro)
@@ -65,7 +65,7 @@
     </collision>
     <inertial>
-      <mass value="1.5"/>
+      <mass value="1.679"/>
       <origin xyz="0.013 0 0.129" rpy="0 0 0"/>
-      <inertia ixx="0.010" ixy="0" ixz="0" iyy="0.010" iyz="0" izz="0.005"/>
+      <inertia ixx="0.050216" ixy="0.000001" ixz="-0.000845" iyy="0.010889" iyz="-0.000001" izz="0.046298"/>
     </inertial>
   </link>
@@ -74,5 +74,5 @@
     <parent link="link_1"/>
     <child  link="link_2"/>
-    <origin xyz="0.024031 0 0.202992" rpy="0 0 0"/>
+    <origin xyz="0.0248 0 0.1443" rpy="0 0 0"/>
     <axis xyz="0 1 0"/>
     <limit lower="-1.6" upper="2.1" effort="20.0" velocity="1.0"/>
@@ -107,5 +107,5 @@
     <parent link="link_2"/>
     <child  link="link_3"/>
-    <origin xyz="-0.015224 0 0.441653" rpy="0 0 0"/>
+    <origin xyz="-0.014494 0 0.442345" rpy="0 0 0"/>
     <axis xyz="0 1 0"/>
     <limit lower="-3.0" upper="0.65" effort="15.0" velocity="1.0"/>
@@ -136,5 +136,5 @@
     <parent link="link_3"/>
     <child  link="link_4"/>
-    <origin xyz="0.119473 0 0.029716" rpy="0 0 0"/>
+    <origin xyz="0.11945 0 0.029736" rpy="0 0 0"/>
     <axis xyz="1 0 0"/>
     <limit lower="-3.1416" upper="3.1416" effort="5.0" velocity="2.0"/>
@@ -165,5 +165,5 @@
     <parent link="link_4"/>
     <child  link="link_5"/>
-    <origin xyz="0.321516 0 0" rpy="0 0 0"/>
+    <origin xyz="0.32345 0 0.09896" rpy="0 0 0"/>
     <axis xyz="0 1 0"/>
     <limit lower="-1.6" upper="1.6" effort="5.0" velocity="2.0"/>
@@ -202,5 +202,5 @@
     <parent link="link_5"/>
     <child  link="link_gripper"/>
-    <origin xyz="0.06 0 0" rpy="0 0 0"/>
+    <origin xyz="0.09432 0 0.0005875" rpy="0 0 0"/>
   </joint>
   <link name="link_gripper">

Commit message: Geometrie du bras corrigee, socle recale, nid re-etiquete
Suite de l'ADR-005, avec NM en session sur la simulation.

URDF — corrections successives, chacune verifiee contre la CAO :
- joint_2 revient a z=0.203 (la valeur 0.1443 de l'URDF livree etait fausse) ;
- joint_5 revient sur l'axe de l'avant-bras (z=0). L'URDF livree le placait 99 mm
  au-dessus ; trois sources independantes le contredisaient : l'emprise du maillage
  (50.5 mm hors matiere), l'axe de symetrie mesure dans le STL (z = 0.03 mm sur 24950
  facettes) et le volume de collision declare par l'URDF elle-meme (cylindre centre sur
  z=0). NM a confirme que l'avant-bras est droit ;
- joint_gripper remonte de 2 mm (0.09432 -> 0.09232) ;
- joint_1 pose sur la face superieure du socle (z=0.02 -> 0).

Consequence : joint_4 ne deplace plus le centre du poignet. L'hypothese qui fonde le
point commande de la teleoperation cartesienne est retablie, et les tests qui disaient
l'inverse sont remis dans le bon sens.

Socle — le maillage livre (assemblage_support.stl, 18726 facettes) remplace l'ancien.
Il est en millimetres, ajoute la platine de montage 261x261 qui manquait, et son point
de reference est celui donne par NM : (-0.5, -111, 203) mm dans le repere du STL est
l'origine du robot. Le socle devient un corps fixe de l'URDF (link "socle") plutot
qu'un maillage orphelin : il suit le robot partout. Les 35 obstacles de la scene
cuisine sont translates du meme deplacement (+0.5, -59.22, -23.9 mm) pour que le socle
reste en contact avec la table.

Nid — RE-ETIQUETAGE. La pose de docking passe de
  [1.5627, 0.9179, 0.4520, 0.0, 0.2009] a [1.56020, 0.93500, 0.58883, -0.00249, 0.04700]
soit [-0.143, +0.980, +7.840, -0.143, -8.818] deg. Elle a ete relevee par NM EN
SIMULATION, en amenant le modele solide du bras dans le berceau apres avoir masque les
robots translucides de MoveIt qui n'affichent pas l'etat reel. NM a decide de ne pas
mesurer sur le robot et de retenir ces valeurs.
Le berceau physique n'a pas bouge : ce sont les angles qui le designent qui changent.
Les poses liees au nid sont decalees du meme delta (sortie du nid, approche_nid,
sortie) ; celles validees par demonstration ne le sont PAS (changeur_outil,
approche_changeur, D_pose_cone, depose_cuisine, D_JOINTS). Deux etiquetages coexistent
donc, comme deja apres le recalage du 2026-09-06, et c'est ecrit en tete des fichiers.

⚠️ Un test reste ROUGE, volontairement :
test_plancher_virtuel_le_bras_glisse_sans_faire_geler_le_garde. Il signale que
POSE_TRAVAIL est desormais 19 mm SOUS son plancher virtuel et a 6 mm du gel de la
garde, parce que Z_SURFACE_CUISINE=0.2916 a ete mesure dans l'ancienne geometrie.
L'assouplir masquerait une marge de securite effondree. C'est la premiere des
constantes cartesiennes a re-mesurer.

Outils — roby_squelette.py : vue de la chaine seule, socle et placements lus dans
l'URDF, trois segments cotes et un triede d'axes etiquete. support_robot.stl avait
toutes ses normales nulles (invisible au rendu, et inutilisable par MoveIt) : elles
sont recalculees, geometrie inchangee.

Co-Authored-By: Claude Opus 5 (1M context) <noreply@anthropic.com>
Claude-Session: https://claude.ai/code/session_0187Ttw7QawW3jcZqaeAZY1B

File: src/neuroneimitationcarote_description/urdf/robot.urdf.xacro (robot description, xacro)
@@ -37,5 +37,7 @@
     <parent link="base_link"/>
     <child  link="link_1"/>
-    <origin xyz="0 0 0.02" rpy="0 0 0"/>
+    <!-- z = 0 : l'axe de base est POSE sur la face superieure du socle, qui affleure
+         exactement l'origine (recalage du 2026-09-20). Valait 0.02 auparavant. -->
+    <origin xyz="0 0 0" rpy="0 0 0"/>
     <axis xyz="0 0 1"/>
     <limit lower="-3.14159" upper="3.14159" effort="10.0" velocity="1.0"/>
@@ -74,5 +76,5 @@
     <parent link="link_1"/>
     <child  link="link_2"/>
-    <origin xyz="0.0248 0 0.1443" rpy="0 0 0"/>
+    <origin xyz="0.0249368 0 0.203" rpy="0 0 0"/>
     <axis xyz="0 1 0"/>
     <limit lower="-1.6" upper="2.1" effort="20.0" velocity="1.0"/>
@@ -165,5 +167,5 @@
     <parent link="link_4"/>
     <child  link="link_5"/>
-    <origin xyz="0.32345 0 0.09896" rpy="0 0 0"/>
+    <origin xyz="0.32345 0 0" rpy="0 0 0"/>
     <axis xyz="0 1 0"/>
     <limit lower="-1.6" upper="1.6" effort="5.0" velocity="2.0"/>
@@ -202,5 +204,5 @@
     <parent link="link_5"/>
     <child  link="link_gripper"/>
-    <origin xyz="0.09432 0 0.0005875" rpy="0 0 0"/>
+    <origin xyz="0.09232 0 0.0005875" rpy="0 0 0"/>
   </joint>
   <link name="link_gripper">
@@ -233,3 +235,36 @@
   </joint>
   <link name="tcp"/>
+  <!-- SOCLE — le support sur lequel le bras est boulonné.
+       Il n'est pas mobile, mais il suit le robot partout où on l'installe : il vit donc
+       dans la description, pas dans une scène. Son maillage est déjà exprimé dans le
+       repère de la base (en-tête du STL), d'où l'origine nulle. Il va de z=-0.179 à
+       z=+0.024, et se pose exactement sur le plateau de la table de la scène cuisine
+       (Table_sous_robot, dessus à z=-0.179).
+       Pas de <collision> : l'ajouter exigerait d'abord de désactiver, dans la SRDF, la
+       collision socle/base_link (adjacents par construction), sinon toute pose devient
+       invalide. Le plateau de la table couvre déjà le volume pour la planification. -->
+  <joint name="joint_socle" type="fixed">
+    <parent link="base_link"/>
+    <child  link="socle"/>
+    <origin xyz="0 0 0" rpy="0 0 0"/>
+  </joint>
+  <link name="socle">
+    <visual>
+      <!-- Maillage livre le 2026-09-20 (assemblage_support.stl) : en MILLIMETRES, et
+           son origine est au point le plus BAS du socle, pas a la base du robot.
+           Point de reference donne par NM : dans le repere du STL, le point
+           (-0.5, -111, 203) mm est celui qui doit coincider avec l'origine du robot
+           et de la scene. C'est le CENTRE de la face superieure de la platine de
+           montage (261 x 261 mm). L'origine ci-dessous est donc simplement l'oppose
+           de ce point, converti en metres.
+           Le decor de la scene cuisine a ete translate du meme deplacement
+           (+0.5, -59.22, -23.9 mm) pour rester en contact avec le socle. -->
+      <origin xyz="0.0005 0.111 -0.203" rpy="0 0 0"/>
+      <geometry>
+        <mesh filename="package://roby_environments/meshes/support_robot.stl"
+              scale="0.001 0.001 0.001"/>
+      </geometry>
+      <material name="dark_grey"/>
+    </visual>
+  </link>
 </robot>
